File: Single_transistor_AMP/AMP/AMP.kicad_pcb (KiCad board)
At the start: 2 copper layers, 0 parts

Commit message: NEW IN LINE
Parts:
- added C1: 0.47uF, Capacitor_THT:C_Disc_D5.0mm_W2.5mm_P5.00mm, F.Cu at (122.4, 127.8)
- added C2: 4.7uF, Capacitor_THT:CP_Radial_D5.0mm_P2.00mm, F.Cu at (132.5, 117.0)
- added C3: 4.7uF, Capacitor_THT:CP_Radial_D4.0mm_P1.50mm, F.Cu at (143.0, 126.2)
- added C4: 47uF, Capacitor_THT:CP_Radial_D5.0mm_P2.00mm, F.Cu at (132.8, 108.0)
- added J1: Audio input, Connector_PinHeader_2.54mm:PinHeader_1x02_P2.54mm_Vertical, F.Cu at (112.0, 119.9)
- added J2: 9 V, Connector_PinHeader_2.54mm:PinHeader_1x02_P2.54mm_Vertical, F.Cu at (112.0, 112.5)
- added LS1: 8ohm, Connector_PinHeader_2.54mm:PinHeader_1x02_P2.54mm_Vertical, F.Cu at (150.9, 117.9)
- added Q1: 2N3904, Package_TO_SOT_THT:TO-92_Inline, F.Cu at (130.6, 127.0)
- added Q2: 2N3904, Package_TO_SOT_THT:TO-92_Inline, F.Cu at (137.4, 127.0)
- added R1: 220k, Resistor_THT:R_Axial_DIN0207_L6.3mm_D2.5mm_P15.24mm_Horizontal, F.Cu at (127.0, 122.7)
- added R2: 27k, Resistor_THT:R_Axial_DIN0207_L6.3mm_D2.5mm_P15.24mm_Horizontal, F.Cu at (117.5, 122.6)
- added R3: 1k, Resistor_THT:R_Axial_DIN0207_L6.3mm_D2.5mm_P15.24mm_Horizontal, F.Cu at (138.9, 106.7)
- added R4: 1k5, Resistor_THT:R_Axial_DIN0207_L6.3mm_D2.5mm_P15.24mm_Horizontal, F.Cu at (122.3, 122.5)
- added R5: 1k, Resistor_THT:R_Axial_DIN0207_L6.3mm_D2.5mm_P15.24mm_Horizontal, F.Cu at (143.3, 121.9)
Routing:
- net Net-(C4-Pad2): track 0.00 -> 63.2 mm
- net Net-(C1-Pad1): track 0.00 -> 35.4 mm
- net Net-(C2-Pad2): track 0.00 -> 22.6 mm
- net Net-(Q1-Pad3): track 0.00 -> 17.7 mm
- net Net-(C3-Pad2): track 0.00 -> 14.4 mm
- net Net-(C3-Pad1): track 0.00 -> 11.0 mm
- net Net-(C1-Pad2): track 0.00 -> 7.62 mm
- added copper zone on B.Cu, net (none)
- added copper zone on F.Cu, net GNDREF
Other:
- board outline added: 44.2 x 26.7 mm
